File: srom/srom.kicad_pcb (KiCad board)
At the start: 2 copper layers, 83.3 x 76.1 mm, 31 parts, among them J1 Conn_01x03_Female, Q1 PMBT2222A, SW1 SW_SPST, U1 4075, U2 74LS245, U3 74LS245, U4 74LS245, U5 Pico-rp2040

Commit message: create v1.3 pcb with switch casing grounded, circuit is unchanged. kicad v8 automatic update at this point
Connections:
- SW1 pad : (no net) -> GND
Other:
- board text added: "github.com/derekfountain/zx-spectrum-pico-rom v1.3"
- board text removed: "github.com/derekfountain/zx-spectrum-pico-rom v1.2"
